File: PCB Rev 2/VolumetricDisplay.kicad_pcb (KiCad board)
At the start: 4 copper layers, 48.5 x 56 mm, 149 parts, among them J1 USB_C_Receptacle_USB2.0_16P, J2 Conn_ARM_SWD_TagConnect_TC2030, Q1 DMN32D2LDF, Q2 DMN32D2LDF, Q3 DMN32D2LDF, Q4 DMN32D2LDF, SW4 TS-1088-AR02016, SW5 TS-1088-AR02016, U2 NCP718xSN330, U3 RP2354B, U4 DRV8311S, U5 DRV5055A1xDBZxQ1, Y1 Abracon ABM8-272-T3

Commit message: Added GND & 3V3 Pours
Made In1 and In2 GND and 3V3 Pours and added some vias and connections for them
Connections:
- D41 pad 2: LED5 -> GND
- D42 pad 2: LED5 -> GND
- D43 pad 2: LED5 -> GND
- D44 pad 2: LED5 -> GND
- D45 pad 2: LED5 -> GND
- D46 pad 2: LED5 -> GND
- D47 pad 2: LED5 -> GND
- D48 pad 2: LED5 -> GND
Routing:
- net GND: track 4.29 -> 70.9 mm, vias 0 -> 7
- net LED6: track 0.00 -> 38.5 mm
- net LED7: track 0.00 -> 38.5 mm
- net LED4: track 0.00 -> 38.5 mm
- net LED2: track 0.00 -> 38.5 mm
- net LED1: track 0.00 -> 38.5 mm
- net LED0: track 0.12 -> 38.6 mm
- net LED3: track 0.00 -> 38.5 mm
- net /MCU/VBUS: track 0.00 -> 14.2 mm
- net Net-(J1-CC1): track 0.00 -> 11.3 mm
- net Net-(J1-CC2): track 0.42 -> 6.72 mm
- net Net-(D1-K): track 0.00 -> 6.08 mm
- net 5V: track 18.8 -> 22.2 mm
- net 3V3: track 2.08 -> 5.19 mm, vias 0 -> 1
- net D_P: track 0.63 -> 2.34 mm
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- added copper zone on In2.Cu, net 3V3
- added copper zone on In1.Cu, net GND
- removed copper zone on In1.Cu, net /MCU/VBUS
